File: PCB/Klave.kicad_pcb (KiCad board)
At the start: 2 copper layers, 32 parts, among them SW1 0:0, SW10 1:3, SW11 1:4, SW12 1:5, SW13 2:0, SW14 2:1, SW15 2:2, SW16 2:3, SW17 2:4, SW18 2:5, SW19 3:0, SW2 0:1, SW20 3:1, SW21 3:2, SW22 3:3, SW23 3:4, SW24 3:5, SW26 4:1, SW27 4:2, SW28 4:3, SW29 4:4, SW3 0:2, SW30 4:5, SW35 5:4, SW36 5:5, SW4 0:3, SW5 0:4, SW6 0:5, SW7 1:0, SW8 1:1, SW9 1:2

Commit message: Create first PCB prototype
Parts:
- added D1: 0:0, KlaveLib:D_SOD-123, F.Cu at (38.0, 54.6)
- added D10: 1:3, KlaveLib:D_SOD-123, F.Cu at (95.0, 52.7)
- added D11: 1:4, KlaveLib:D_SOD-123, F.Cu at (114.0, 60.3)
- added D12: 1:5, KlaveLib:D_SOD-123, F.Cu at (133.0, 62.2)
- added D13: 2:0, KlaveLib:D_SOD-123, F.Cu at (38.0, 92.6)
- added D14: 2:1, KlaveLib:D_SOD-123, F.Cu at (57.0, 90.7)
- added D15: 2:2, KlaveLib:D_SOD-123, F.Cu at (76.0, 76.5)
- added D16: 2:3, KlaveLib:D_SOD-123, F.Cu at (95.0, 71.7)
- added D17: 2:4, KlaveLib:D_SOD-123, F.Cu at (114.0, 79.3)
- added D18: 2:5, KlaveLib:D_SOD-123, F.Cu at (133.0, 81.2)
- added D19: 3:0, KlaveLib:D_SOD-123, F.Cu at (38.0, 111.6)
- added D2: 0:1, KlaveLib:D_SOD-123, F.Cu at (57.0, 52.7)
- added D20: 3:1, KlaveLib:D_SOD-123, F.Cu at (57.0, 109.7)
- added D21: 3:2, KlaveLib:D_SOD-123, F.Cu at (76.0, 95.5)
- added D22: 3:3, KlaveLib:D_SOD-123, F.Cu at (95.0, 90.7)
- added D23: 3:4, KlaveLib:D_SOD-123, F.Cu at (114.0, 98.3)
- added D24: 3:5, KlaveLib:D_SOD-123, F.Cu at (133.0, 100.2)
- added D26: 4:1, KlaveLib:D_SOD-123, F.Cu at (84.5, 117.3)
- added D27: 4:2, KlaveLib:D_SOD-123, F.Cu at (103.5, 117.3)
- added D28: 4:3, KlaveLib:D_SOD-123, F.Cu at (125.4, 120.2)
- added D29: 4:4, KlaveLib:D_SOD-123, F.Cu at (155.0, 111.0)
- added D3: 0:2, KlaveLib:D_SOD-123, F.Cu at (76.0, 38.5)
- added D30: 4:5, KlaveLib:D_SOD-123, F.Cu at (171.5, 120.2)
- added D31: 5:0, KlaveLib:D_SOD-123, F.Cu at (157.5, 92.2)
- added D36: 5:5, KlaveLib:D_SOD-123, F.Cu at (162.4, 136.8)
- added D4: 0:3, KlaveLib:D_SOD-123, F.Cu at (95.0, 33.7)
- added D5: 0:4, KlaveLib:D_SOD-123, F.Cu at (114.0, 41.3)
- added D6: 0:5, KlaveLib:D_SOD-123, F.Cu at (133.0, 43.2)
- added D7: 1:0, KlaveLib:D_SOD-123, F.Cu at (38.0, 73.6)
- added D8: 1:1, KlaveLib:D_SOD-123, F.Cu at (57.0, 71.7)
- added D9: 1:2, KlaveLib:D_SOD-123, F.Cu at (76.0, 57.5)
- added Dr: 5:4, KlaveLib:D_SOD-123, F.Cu at (145.8, 127.8)
- added J1: 6P6C, KlaveLib:RJ12_6P6C, F.Cu at (165.4, 56.8)
- added J2: OLED, KlaveLib:Display_OLED_128x32, F.Cu at (149.1, 76.2)
- added JP1: Front, Jumper:SolderJumper-2_P1.3mm_Open_Pad1.0x1.5mm, F.Cu at (149.1, 72.4)
- added JP2: Front, Jumper:SolderJumper-2_P1.3mm_Open_Pad1.0x1.5mm, F.Cu at (151.6, 72.4)
- added JP3: Front, Jumper:SolderJumper-2_P1.3mm_Open_Pad1.0x1.5mm, F.Cu at (154.2, 72.4)
- added JP4: Front, Jumper:SolderJumper-2_P1.3mm_Open_Pad1.0x1.5mm, F.Cu at (156.7, 72.4)
- added JP5: Back, Jumper:SolderJumper-2_P1.3mm_Open_Pad1.0x1.5mm, B.Cu at (156.7, 72.4)
- added JP6: Back, Jumper:SolderJumper-2_P1.3mm_Open_Pad1.0x1.5mm, B.Cu at (154.2, 72.4)
- added JP7: Back, Jumper:SolderJumper-2_P1.3mm_Open_Pad1.0x1.5mm, B.Cu at (151.6, 72.4)
- added JP8: Back, Jumper:SolderJumper-2_P1.3mm_Open_Pad1.0x1.5mm, B.Cu at (149.1, 72.4)
- added R1: 4k7, KlaveLib:R_1206_3216Metric, F.Cu at (152.9, 50.8)
- added R2: 4k7, KlaveLib:R_1206_3216Metric, F.Cu at (152.9, 53.3)
- added R3: 47, KlaveLib:R_1206_3216Metric, F.Cu at (151.4, 45.8)
- added R4: 47, KlaveLib:R_1206_3216Metric, F.Cu at (154.4, 45.8)
- added R5: 10, KlaveLib:R_1206_3216Metric, F.Cu at (152.8, 60.4)
- added SW0: Reset, KlaveLib:SW_Tactile_2pin, F.Cu at (152.9, 80.1)
- added U1: ProMicro, KlaveLib:Arduino_ProMicro, F.Cu at (152.9, 53.3)
Routing:
- net col0: track 0.00 -> 256.1 mm, vias 0 -> 5
- net col1: track 0.00 -> 224.1 mm, vias 0 -> 5
- net col2: track 0.00 -> 207.6 mm, vias 0 -> 5
- net col3: track 0.00 -> 196.1 mm, vias 0 -> 5
- net row3: track 0.00 -> 195.1 mm, vias 0 -> 7
- net col4: track 0.00 -> 192.3 mm, vias 0 -> 6
- net row0: track 0.00 -> 191.4 mm, vias 0 -> 8
- net col5: track 0.00 -> 182.2 mm, vias 0 -> 8
- net row1: track 0.00 -> 181.1 mm, vias 0 -> 9
- net row2: track 0.00 -> 176.0 mm, vias 0 -> 10
- net row4: track 0.00 -> 169.4 mm, vias 0 -> 7
- net GND: track 0.00 -> 129.1 mm, vias 0 -> 2
- net row5: track 0.00 -> 110.3 mm, vias 0 -> 7
- net VCC: track 0.00 -> 59.3 mm, vias 0 -> 2
- net SDA: track 0.00 -> 53.7 mm, vias 0 -> 3
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