File: PCB/Klave.kicad_pcb (KiCad board)
At the start: 2 copper layers, 156.3 x 127.5 mm, 87 parts, among them J1 6P6C, J2 OLED, SW0 Reset, SW1 0:0, SW10 1:3, SW11 1:4, SW12 1:5, SW13 2:0, SW14 2:1, SW15 2:2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

Commit message: Add more vias
Routing:
- net GND: vias 82 -> 102
